File: asd_pa_1/poweramp.sch (KiCad schematic (older format))
At the start: 55 parts, among them P1 CONN_01X02, P2 CONN_01X03, P3 CONN_01X02, P4 CONN_01X01, P5 CONN_01X01, Q1 BC556, Q10 BC546, Q11 MJE243C, Q12 MJE253C, Q13 MJL21194C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

Commit message: Updated schematics and PCB.  Removed some minor errors with the first prototype.
Parts:
- C1, C2, C3, C4, C6, C8: symbol C -> C-RESCUE-poweramp
- C5, C7, C9: symbol CP1 -> CP1-RESCUE-poweramp
- D1: symbol ZENER -> ZENER-RESCUE-poweramp
- R1, R10, R11, R12, R13, R14, R15, R16, R17, R18, R19, R2, R20, R21, R3, R4, R5, R6, R7, R8, R9: symbol R -> R-RESCUE-poweramp
- XRV1: symbol POT -> POT-RESCUE-poweramp
Changed lines of the file:
@@
 EESchema Schematic File Version 2
+LIBS:poweramp-rescue
 LIBS:power
 LIBS:device
@@
 LIBS:memory
 LIBS:xilinx
-LIBS:special
 LIBS:microcontrollers
 LIBS:dsp
@@
 $EndComp
 $Comp
-L CP1 C5
+L CP1-RESCUE-poweramp C5
 U 1 1 54189F9D
 P 6650 2450
@@
 $EndSheet
 $Comp
-L R R21
+L R-RESCUE-poweramp R21
 U 1 1 5414600A
 P 7800 3700
@@
 $EndComp
 $Comp
-L R R20
+L R-RESCUE-poweramp R20
 U 1 1 54142FD1
 P 7800 2800
@@
 $EndComp
 $Comp
-L VEE #PWR11
+L VEE #PWR01
 U 1 1 5412EC89
 P 8600 3550
-F 0 "#PWR11" H 8600 3750 40  0001 C CNN
+F 0 "#PWR01" H 8600 3750 40  0001 C CNN
 F 1 "VEE" H 8600 3700 40  0000 C CNN
 F 2 "" H 8600 3550 60  0001 C CNN
@@
 gnd_z
 $Comp
-L VCC #PWR01
+L VCC #PWR02
 U 1 1 5411E822
 P 8600 3450
-F 0 "#PWR01" H 8600 3550 30  0001 C CNN
+F 0 "#PWR02" H 8600 3550 30  0001 C CNN
 F 1 "VCC" H 8600 3575 30  0000 C CNN
 F 2 "" H 8600 3450 60  0001 C CNN
@@
 gnd_dc
 $Comp
-L R R2
+L R-RESCUE-poweramp R2
 U 1 1 5406EDC1
 P 2200 4850
@@
 $EndComp
 $Comp
-L VEE #PWR13
+L VEE #PWR03
 U 1 1 5406C496
 P 10150 1150
-F 0 "#PWR13" H 10150 1350 40  0001 C CNN
+F 0 "#PWR03" H 10150 1350 40  0001 C CNN
 F 1 "VEE" H 10150 1300 40  0000 C CNN
 F 2 "" H 10150 1150 60  0001 C CNN
@@
 $EndComp
 $Comp
-L VCC #PWR02
+L VCC #PWR04
 U 1 1 5406C48B
 P 8950 1150
-F 0 "#PWR02" H 8950 1250 30  0001 C CNN
+F 0 "#PWR04" H 8950 1250 30  0001 C CNN
 F 1 "VCC" H 8950 1275 30  0000 C CNN
 F 2 "" H 8950 1150 60  0001 C CNN
@@
 $EndComp
 $Comp
-L CP1 C9
+L CP1-RESCUE-poweramp C9
 U 1 1 5406C472
 P 10150 1550
@@
 $EndComp
 $Comp
-L CP1 C7
+L CP1-RESCUE-poweramp C7
 U 1 1 5406C45C
 P 9350 1550
@@
 $EndComp
 $Comp
-L GND #PWR03
+L GND #PWR05
 U 1 1 5406C202
 P 2250 2150
-F 0 "#PWR03" H 2250 2150 30  0001 C CNN
+F 0 "#PWR05" H 2250 2150 30  0001 C CNN
 F 1 "GND" H 2250 2080 30  0001 C CNN
 F 2 "" H 2250 2150 60  0001 C CNN
@@
 $EndComp
 $Comp
-L VEE #PWR2
+L VEE #PWR06
 U 1 1 5406C1EB
 P 2000 1400
-F 0 "#PWR2" H 2000 1600 40  0001 C CNN
+F 0 "#PWR06" H 2000 1600 40  0001 C CNN
 F 1 "VEE" H 2000 1550 40  0000 C CNN
 F 2 "" H 2000 1400 60  0001 C CNN
@@
 $EndComp
 $Comp
-L VCC #PWR04
+L VCC #PWR07
 U 1 1 5406C1D1
 P 2000 1100
-F 0 "#PWR04" H 2000 1200 30  0001 C CNN
+F 0 "#PWR07" H 2000 1200 30  0001 C CNN
 F 1 "VCC" H 2000 1225 30  0000 C CNN
 F 2 "" H 2000 1100 60  0001 C CNN
@@
 $EndComp
 $Comp
-L GND #PWR05
+L GND #PWR08
 U 1 1 5406BAED
 P 5900 4600
-F 0 "#PWR05" H 5900 4600 30  0001 C CNN
+F 0 "#PWR08" H 5900 4600 30  0001 C CNN
 F 1 "GND" H 5900 4530 30  0001 C CNN
 F 2 "" H 5900 4600 60  0001 C CNN
@@
 $EndComp
 $Comp
-L GND #PWR06
+L GND #PWR09
 U 1 1 54062520
 P 2200 5250
-F 0 "#PWR06" H 2200 5250 30  0001 C CNN
+F 0 "#PWR09" H 2200 5250 30  0001 C CNN
 F 1 "GND" H 2200 5180 30  0001 C CNN
 F 2 "" H 2200 5250 60  0001 C CNN
@@
 $EndComp
 $Comp
-L GND #PWR07
+L GND #PWR010
 U 1 1 540624E7
 P 5400 2250
-F 0 "#PWR07" H 5400 2250 30  0001 C CNN
+F 0 "#PWR010" H 5400 2250 30  0001 C CNN
 F 1 "GND" H 5400 2180 30  0001 C CNN
 F 2 "" H 5400 2250 60  0001 C CNN
@@
 $EndComp
 $Comp
-L GND #PWR08
+L GND #PWR011
 U 1 1 540624C2
 P 3150 2450
-F 0 "#PWR08" H 3150 2450 30  0001 C CNN
+F 0 "#PWR011" H 3150 2450 30  0001 C CNN
 F 1 "GND" H 3150 2380 30  0001 C CNN
 F 2 "" H 3150 2450 60  0001 C CNN
@@
 $EndComp
 $Comp
-L VEE #PWR8
+L VEE #PWR012
 U 1 1 54062385
 P 5600 6000
-F 0 "#PWR8" H 5600 6200 40  0001 C CNN
+F 0 "#PWR012" H 5600 6200 40  0001 C CNN
 F 1 "VEE" H 5600 6150 40  0000 C CNN
 F 2 "" H 5600 6000 60  0001 C CNN
@@
 $EndComp
 $Comp
-L VCC #PWR09
+L VCC #PWR013
 U 1 1 540622E5
 P 5200 750
-F 0 "#PWR09" H 5200 850 30  0001 C CNN
+F 0 "#PWR013" H 5200 850 30  0001 C CNN
 F 1 "VCC" H 5200 875 30  0000 C CNN
 F 2 "" H 5200 750 60  0001 C CNN
@@
 gnd_z
 $Comp
-L R R19
+L R-RESCUE-poweramp R19
 U 1 1 53D77405
 P 7250 3700
@@
 $EndComp
 $Comp
-L R R3
+L R-RESCUE-poweramp R3
 U 1 1 53D6ACF1
 P 2800 4200
@@
 $EndComp
 $Comp
-L C C2
+L C-RESCUE-poweramp C2
 U 1 1 53D6ACE3
 P 2500 3900
@@
 $EndComp
 $Comp
-L C C1
+L C-RESCUE-poweramp C1
 U 1 1 53D6AC9C
 P 2200 4200
@@
 $EndComp
 $Comp
-L R R1
+L R-RESCUE-poweramp R1
 U 1 1 53D6AC8E
 P 1900 3900
@@
 $EndComp
 $Comp
-L C C3
+L C-RESCUE-poweramp C3
 U 1 1 53D6AA3C
 P 4750 2950
@@
 $EndComp
 $Comp
-L C C4
+L C-RESCUE-poweramp C4
 U 1 1 53D668B4
 P 5950 4200
@@
 $EndComp
 $Comp
-L R R10
+L R-RESCUE-poweramp R10
 U 1 1 53D66553
 P 4750 3500
@@
 $EndComp
 $Comp
-L R R11
+L R-RESCUE-poweramp R11
 U 1 1 53D66541
 P 5200 3900
@@
 $EndComp
 $Comp
-L R R18
+L R-RESCUE-poweramp R18
 U 1 1 53D663F4
 P 7250 2800
@@
 $EndComp
 $Comp
-L R R12
+L R-RESCUE-poweramp R12
 U 1 1 53D65D85
 P 5400 1900
@@
 $EndComp
 $Comp
-L R R16
+L R-RESCUE-poweramp R16
 U 1 1 53D65D52
 P 6300 1050
@@
 $EndComp
 $Comp
-L POT XRV1
+L POT-RESCUE-poweramp XRV1
 U 1 1 53D64F58
 P 5800 2750
@@
 $EndComp
 $Comp
-L R R7
+L R-RESCUE-poweramp R7
 U 1 1 53D64821
 P 3850 1200
@@
 $EndComp
 $Comp
-L R R15
+L R-RESCUE-poweramp R15
 U 1 1 53D63E01
 P 6000 3300
@@
 $EndComp
 $Comp
-L R R14
+L R-RESCUE-poweramp R14
 U 1 1 53D63D1B
 P 5800 2150
@@
 $EndComp
 $Comp
-L R R4
+L R-RESCUE-poweramp R4
 U 1 1 53D63D10
 P 3150 2100
@@
 $EndComp
 $Comp
-L ZENER D1
+L ZENER-RESCUE-poweramp D1
 U 1 1 53D63CFF
 P 3150 1300
@@
 $EndComp
 $Comp
-L R R17
+L R-RESCUE-poweramp R17
 U 1 1 53D63CA1
 P 6300 5450
@@
 $EndComp
 $Comp
-L R R13
+L R-RESCUE-poweramp R13
 U 1 1 53D63C98
 P 5600 5450
@@
 $EndComp
 $Comp
-L R R9
+L R-RESCUE-poweramp R9
 U 1 1 53D63BCA
 P 4250 5450
@@
 $EndComp
 $Comp
-L R R6
+L R-RESCUE-poweramp R6
 U 1 1 53D63BC4
 P 3450 5450
@@
 $EndComp
 $Comp
-L R R8
+L R-RESCUE-poweramp R8
 U 1 1 53D63B6E
 P 4250 3400
@@
 $EndComp
 $Comp
-L R R5
+L R-RESCUE-poweramp R5
 U 1 1 53D63B5B
 P 3450 3400
@@
 $EndComp
 $Comp
-L C C6
+L C-RESCUE-poweramp C6
 U 1 1 5436F4FD
 P 8950 1550
@@
 $EndComp
 $Comp
-L C C8
+L C-RESCUE-poweramp C8
 U 1 1 5436FAA2
 P 9750 1550
