File: asd_pre_1/pcb/EFM32GG.sch (KiCad schematic (older format))
At the start: 32 parts, among them P1 SD_Card_DM1, P14 MCU Debug, P6 GPIO, P7 Mute, P8 LEDs, P9 Volume, U1 EFM32GG232F1024, X1 48MHz

Commit message: Updated schematics and PCB.  Removed some minor errors with the first prototype.
Parts:
- C1, C12, C2, C4, C5, C6, C7, C8, C9: symbol C -> C-RESCUE-preamp
- C10, C11, C3: symbol CP1 -> CP1-RESCUE-preamp
- R1, R10, R11, R12, R2, R3, R4, R5, R6, R7, R8, R9: symbol R -> R-RESCUE-preamp
Changed lines of the file:
@@
 EESchema Schematic File Version 2
+LIBS:preamp-rescue
 LIBS:power
 LIBS:device
@@
 LIBS:memory
 LIBS:xilinx
-LIBS:special
 LIBS:microcontrollers
 LIBS:dsp
@@
 encoding utf-8
 Sheet 2 9
-Title ""
+Title "AsD Pre 1 Digital Preamplifier -- MCU"
 Date ""
 Rev ""
-Comp ""
+Comp "Asbjørn Djupdal"
 Comment1 ""
 Comment2 ""
@@
 $EndComp
 $Comp
-L CP1 C10
+L CP1-RESCUE-preamp C10
 U 1 1 5464FC3A
 P 4600 1625
@@
 $EndComp
 $Comp
-L C C9
+L C-RESCUE-preamp C9
 U 1 1 5464FD6F
 P 4300 1625
@@
 $EndComp
 $Comp
-L C C8
+L C-RESCUE-preamp C8
 U 1 1 5464FDFA
 P 4050 1625
@@
 $EndComp
 $Comp
-L C C6
+L C-RESCUE-preamp C6
 U 1 1 5464FE1B
 P 3800 1625
@@
 $EndComp
 $Comp
-L C C5
+L C-RESCUE-preamp C5
 U 1 1 5464FE3D
 P 3550 1625
@@
 $EndComp
 $Comp
-L CP1 C3
+L CP1-RESCUE-preamp C3
 U 1 1 5464FFDB
 P 3350 1025
@@
 $EndComp
 $Comp
-L C C1
+L C-RESCUE-preamp C1
 U 1 1 54650587
 P 900 1725
@@
 $EndComp
 $Comp
-L C C2
+L C-RESCUE-preamp C2
 U 1 1 546505F2
 P 1200 1725
@@
 $EndComp
 $Comp
-L R R4
+L R-RESCUE-preamp R4
 U 1 1 54670F14
 P 8450 1900
@@
 $EndComp
 $Comp
-L R R6
+L R-RESCUE-preamp R6
 U 1 1 54670FE7
 P 8625 1900
@@
 $EndComp
 $Comp
-L R R12
+L R-RESCUE-preamp R12
 U 1 1 5467101C
 P 9175 1900
@@
 $EndComp
 $Comp
-L R R10
+L R-RESCUE-preamp R10
 U 1 1 54671054
 P 8900 3450
@@
 $EndComp
 $Comp
-L R R9
+L R-RESCUE-preamp R9
 U 1 1 546711DB
 P 8900 3275
@@
 $EndComp
 $Comp
-L R R8
+L R-RESCUE-preamp R8
 U 1 1 54671209
 P 8900 3050
@@
 $EndComp
 $Comp
-L R R7
+L R-RESCUE-preamp R7
 U 1 1 54671258
 P 8900 2850
@@
 $EndComp
 $Comp
-L C C12
+L C-RESCUE-preamp C12
 U 1 1 5467480C
 P 8050 1875
@@
 $EndComp
 $Comp
-L CP1 C11
+L CP1-RESCUE-preamp C11
 U 1 1 54674E07
 P 7725 1875
@@
 M0
 $Comp
-L R R11
+L R-RESCUE-preamp R11
 U 1 1 54815CD9
 P 9050 5600
@@
 $EndComp
 $Comp
-L C C7
+L C-RESCUE-preamp C7
 U 1 1 547FBCC0
 P 3950 4975
@@
 $EndComp
 $Comp
-L C C4
+L C-RESCUE-preamp C4
 U 1 1 547FBCC6
 P 3350 4975
@@
 I2C0_SDA
 $Comp
-L R R1
+L R-RESCUE-preamp R1
 U 1 1 547FBD08
 P 3500 3075
@@
 $EndComp
 $Comp
-L R R2
+L R-RESCUE-preamp R2
 U 1 1 547FBD0E
 P 3700 3075
@@
 $EndComp
 $Comp
-L R R5
+L R-RESCUE-preamp R5
 U 1 1 5482E5ED
 P 8600 5700
@@
 Connection ~ 6375 5700
 $Comp
-L R R3
+L R-RESCUE-preamp R3
 U 1 1 5483D977
 P 8150 5800
