File: asd_pre_1/pcb/adc.sch (KiCad schematic (older format))
At the start: 54 parts, among them P10 LIN, P11 RIN, U15 LM4562, U16 LM4562, U17 SD103ASDM, U18 SD103ASDM, U19 cs5361

Commit message: Updated schematics and PCB.  Removed some minor errors with the first prototype.
Parts:
- C127, C128, C133, C134, C135, C136, C137, C138, C139, C140, C141, C142, C143, C144, C145, C146, C147, C148, C149, C150, C151, C152, C153: symbol C -> C-RESCUE-preamp
- C129, C130, C131, C132: symbol CP1 -> CP1-RESCUE-preamp
- R54, R55, R56, R57, R58, R59, R60, R61, R62, R63, R64, R65, R66, R67, R68, R69, R70, R71, R72, R73: symbol R -> R-RESCUE-preamp
