File: asd_pre_1/pcb/dac.sch (KiCad schematic (older format))
At the start: 42 parts, among them P12 LOUT, P13 ROUT, U4 CS4398, U5 LM4562

Commit message: Updated schematics and PCB.  Removed some minor errors with the first prototype.
Parts:
- C21, C22, C23, C25, C27, C28, C29, C31, C34, C35, C36, C37, C38, C39, C40, C41, C42, C43: symbol C -> C-RESCUE-preamp
- C24, C26, C30, C32, C33: symbol CP1 -> CP1-RESCUE-preamp
- R16, R17, R18, R19, R20, R21, R22, R23, R24, R25, R26, R27, R28, R29, R30: symbol R -> R-RESCUE-preamp
Changed lines of the file:
@@
 EESchema Schematic File Version 2
+LIBS:preamp-rescue
 LIBS:power
 LIBS:device
@@
 LIBS:memory
 LIBS:xilinx
-LIBS:special
 LIBS:microcontrollers
 LIBS:dsp
@@
 encoding utf-8
 Sheet 4 9
-Title ""
+Title "AsD Pre 1 Digital Preamplifier -- DAC"
 Date ""
 Rev ""
-Comp ""
+Comp "Asbjørn Djupdal"
 Comment1 ""
 Comment2 ""
@@
 $EndComp
 $Comp
-L C C23
+L C-RESCUE-preamp C23
 U 1 1 54688BFB
 P 1575 6825
@@
 $EndComp
 $Comp
-L CP1 C24
+L CP1-RESCUE-preamp C24
 U 1 1 54688E26
 P 1850 6825
@@
 $EndComp
 $Comp
-L C C25
+L C-RESCUE-preamp C25
 U 1 1 54688EF9
 P 2375 6825
@@
 $EndComp
 $Comp
-L CP1 C26
+L CP1-RESCUE-preamp C26
 U 1 1 546891DE
 P 2650 6825
@@
 $EndComp
 $Comp
-L CP1 C33
+L CP1-RESCUE-preamp C33
 U 1 1 54689475
 P 5775 3200
@@
 $EndComp
 $Comp
-L C C29
+L C-RESCUE-preamp C29
 U 1 1 5468953D
 P 4575 3200
@@
 $EndComp
 $Comp
-L CP1 C30
+L CP1-RESCUE-preamp C30
 U 1 1 5468969E
 P 4825 3200
@@
 $EndComp
 $Comp
-L C C31
+L C-RESCUE-preamp C31
 U 1 1 5468982C
 P 5200 3200
@@
 $EndComp
 $Comp
-L CP1 C32
+L CP1-RESCUE-preamp C32
 U 1 1 54689871
 P 5450 3200
@@
 $EndComp
 $Comp
-L C C22
+L C-RESCUE-preamp C22
 U 1 1 5467D927
 P 1350 6825
@@
 $EndComp
 $Comp
-L C C21
+L C-RESCUE-preamp C21
 U 1 1 5467D95A
 P 1125 6825
@@
 $EndComp
 $Comp
-L C C27
+L C-RESCUE-preamp C27
 U 1 1 54687F74
 P 3375 6825
@@
 $EndComp
 $Comp
-L C C28
+L C-RESCUE-preamp C28
 U 1 1 54688051
 P 3700 6825
@@
 $EndComp
 $Comp
-L R R16
+L R-RESCUE-preamp R16
 U 1 1 547D943A
 P 2525 3700
@@
 nRST
 $Comp
-L R R17
+L R-RESCUE-preamp R17
 U 1 1 5486BC58
 P 6675 1875
@@
 $EndComp
 $Comp
-L R R23
+L R-RESCUE-preamp R23
 U 1 1 5486BD57
 P 7225 1875
@@
 $EndComp
 $Comp
-L C C34
+L C-RESCUE-preamp C34
 U 1 1 5486BDAD
 P 6950 2100
@@
 $EndComp
 $Comp
-L C C35
+L C-RESCUE-preamp C35
 U 1 1 5486BE34
 P 6950 2550
@@
 $EndComp
 $Comp
-L R R18
+L R-RESCUE-preamp R18
 U 1 1 5486C150
 P 6675 2775
@@
 $EndComp
 $Comp
-L R R24
+L R-RESCUE-preamp R24
 U 1 1 5486C1D2
 P 7225 2775
@@
 $EndComp
 $Comp
-L C C40
+L C-RESCUE-preamp C40
 U 1 1 5486CB19
 P 7750 1400
@@
 $EndComp
 $Comp
-L R R27
+L R-RESCUE-preamp R27
 U 1 1 5486CDA1
 P 7800 1175
@@
 Connection ~ 8700 1400
 $Comp
-L R R21
+L R-RESCUE-preamp R21
 U 1 1 5486D731
 P 6950 3050
@@
 $EndComp
 $Comp
-L C C38
+L C-RESCUE-preamp C38
 U 1 1 5486D897
 P 7525 3050
@@
 	8075 2425 8075 2375
 $Comp
-L R R19
+L R-RESCUE-preamp R19
 U 1 1 5486FA46
 P 6675 4275
@@
 $EndComp
 $Comp
-L R R25
+L R-RESCUE-preamp R25
 U 1 1 5486FA4C
 P 7225 4275
@@
 $EndComp
 $Comp
-L C C36
+L C-RESCUE-preamp C36
 U 1 1 5486FA53
 P 6950 4500
@@
 $EndComp
 $Comp
-L C C37
+L C-RESCUE-preamp C37
 U 1 1 5486FA5A
 P 6950 4950
@@
 $EndComp
 $Comp
-L R R20
+L R-RESCUE-preamp R20
 U 1 1 5486FA66
 P 6675 5175
@@
 $EndComp
 $Comp
-L R R26
+L R-RESCUE-preamp R26
 U 1 1 5486FA6C
 P 7225 5175
@@
 $EndComp
 $Comp
-L C C41
+L C-RESCUE-preamp C41
 U 1 1 5486FA73
 P 7750 3800
@@
 $EndComp
 $Comp
-L R R28
+L R-RESCUE-preamp R28
 U 1 1 5486FA79
 P 7800 3575
@@
 Connection ~ 8700 3800
 $Comp
-L R R22
+L R-RESCUE-preamp R22
 U 1 1 5486FA96
 P 6950 5450
@@
 $EndComp
 $Comp
-L C C39
+L C-RESCUE-preamp C39
 U 1 1 5486FA9D
 P 7525 5450
@@
 	9625 4475 9625 4925
 $Comp
-L R R29
+L R-RESCUE-preamp R29
 U 1 1 548734DC
 P 8975 1975
@@
 $EndComp
 $Comp
-L C C42
+L C-RESCUE-preamp C42
 U 1 1 54873709
 P 9250 2200
@@
 Connection ~ 9250 1975
 $Comp
-L R R30
+L R-RESCUE-preamp R30
 U 1 1 54873FA3
 P 8975 4375
@@
 	8675 4375 8725 4375
 $Comp
-L C C43
+L C-RESCUE-preamp C43
 U 1 1 548742C1
 P 9250 4600
