File: asd_pre_1/pcb/eth.sch (KiCad schematic (older format))
At the start: 26 parts, among them P2 RJ45-MAGJACK, U6 ENC424J600, X2 25MHz

Commit message: Updated schematics and PCB.  Removed some minor errors with the first prototype.
Parts:
- C44: symbol CP1 -> CP1-RESCUE-preamp
- C45, C46, C47, C48, C49, C50, C51, C52, C53, C54, C55, C56, C57: symbol C -> C-RESCUE-preamp
- R31, R32, R33, R34, R35, R36, R37, R38, R39: symbol R -> R-RESCUE-preamp
Changed lines of the file:
@@
 EESchema Schematic File Version 2
+LIBS:preamp-rescue
 LIBS:power
 LIBS:device
@@
 LIBS:memory
 LIBS:xilinx
-LIBS:special
 LIBS:microcontrollers
 LIBS:dsp
@@
 encoding utf-8
 Sheet 5 9
-Title ""
+Title "AsD Pre 1 Digital Preamplifier -- Ethernet"
 Date ""
 Rev ""
-Comp ""
+Comp "Asbjørn Djupdal"
 Comment1 ""
 Comment2 ""
@@
 $EndComp
 $Comp
-L C C45
+L C-RESCUE-preamp C45
 U 1 1 5467978D
 P 4100 2125
@@
 $EndComp
 $Comp
-L C C46
+L C-RESCUE-preamp C46
 U 1 1 54679887
 P 4750 2125
@@
 $EndComp
 $Comp
-L C C51
+L C-RESCUE-preamp C51
 U 1 1 5467C4C9
 P 8375 1525
@@
 $EndComp
 $Comp
-L C C52
+L C-RESCUE-preamp C52
 U 1 1 5467C80A
 P 8600 1525
@@
 $EndComp
 $Comp
-L C C53
+L C-RESCUE-preamp C53
 U 1 1 5467C83F
 P 8825 1525
@@
 $EndComp
 $Comp
-L C C54
+L C-RESCUE-preamp C54
 U 1 1 5467C873
 P 9050 1525
@@
 $EndComp
 $Comp
-L C C55
+L C-RESCUE-preamp C55
 U 1 1 5467C8A8
 P 9275 1525
@@
 $EndComp
 $Comp
-L C C56
+L C-RESCUE-preamp C56
 U 1 1 5467C8DE
 P 9500 1525
@@
 $EndComp
 $Comp
-L C C57
+L C-RESCUE-preamp C57
 U 1 1 5467C940
 P 9725 1525
@@
 $EndComp
 $Comp
-L CP1 C44
+L CP1-RESCUE-preamp C44
 U 1 1 5467D7EB
 P 2000 3075
@@
 	2000 3275 2000 3325
 $Comp
-L R R32
+L R-RESCUE-preamp R32
 U 1 1 5467DBCD
 P 4075 3550
@@
 	4075 3825 4075 3800
 $Comp
-L R R33
+L R-RESCUE-preamp R33
 U 1 1 5467EAA1
 P 5350 2900
@@
 $EndComp
 $Comp
-L R R34
+L R-RESCUE-preamp R34
 U 1 1 5467EC0F
 P 5350 3475
@@
 $EndComp
 $Comp
-L R R35
+L R-RESCUE-preamp R35
 U 1 1 5467F0AF
 P 5350 4175
@@
 $EndComp
 $Comp
-L R R36
+L R-RESCUE-preamp R36
 U 1 1 5467F0B6
 P 5350 4750
@@
 $EndComp
 $Comp
-L C C49
+L C-RESCUE-preamp C49
 U 1 1 5467F116
 P 6000 3250
@@
 $EndComp
 $Comp
-L R R37
+L R-RESCUE-preamp R37
 U 1 1 5467F276
 P 6000 2275
@@
 Connection ~ 5350 4475
 $Comp
-L C C50
+L C-RESCUE-preamp C50
 U 1 1 5467FF77
 P 6275 5375
@@
 $EndComp
 $Comp
-L C C48
+L C-RESCUE-preamp C48
 U 1 1 5468018E
 P 5900 5000
@@
 $EndComp
 $Comp
-L C C47
+L C-RESCUE-preamp C47
 U 1 1 546802F2
 P 5900 3875
@@
 	10050 4475 10100 4475
 $Comp
-L R R38
+L R-RESCUE-preamp R38
 U 1 1 5468214A
 P 7925 4375
@@
 $EndComp
 $Comp
-L R R39
+L R-RESCUE-preamp R39
 U 1 1 54682483
 P 7925 4575
@@
 	1200 3775 2500 3775
 $Comp
-L R R31
+L R-RESCUE-preamp R31
 U 1 1 54682FB8
 P 1600 3425
