File: asd_pre_1/pcb/fpga_power.sch (KiCad schematic (older format))
At the start: 39 parts, among them U9 xc7a100tftg256

Commit message: Updated schematics and PCB.  Removed some minor errors with the first prototype.
Parts:
- C60, C61: symbol CP1 -> CP1-RESCUE-preamp
- C62, C63, C64, C65, C66, C67, C68, C69, C70, C71, C72, C73, C74, C75, C76, C77, C78, C79, C80, C81, C82, C83, C84, C85, C86, C87, C88, C89, C90, C91, C92, C93, C94, C95, C96, C97: symbol C -> C-RESCUE-preamp
Changed lines of the file:
@@
 EESchema Schematic File Version 2
+LIBS:preamp-rescue
 LIBS:power
 LIBS:device
@@
 LIBS:memory
 LIBS:xilinx
-LIBS:special
 LIBS:microcontrollers
 LIBS:dsp
@@
 encoding utf-8
 Sheet 7 9
-Title ""
+Title "AsD Pre 1 Digital Preamplifier"
 Date ""
 Rev ""
-Comp ""
+Comp "Asbjørn Djupdal"
 Comment1 ""
 Comment2 ""
@@
 $EndComp
 $Comp
-L +1.0V #PWR076
+L +1.0V #PWR075
 U 1 1 5479DBB4
 P 3200 1725
-F 0 "#PWR076" H 3200 1865 20  0001 C CNN
+F 0 "#PWR075" H 3200 1865 20  0001 C CNN
 F 1 "+1.0V" H 3200 1835 30  0000 C CNN
 F 2 "" H 3200 1725 60  0000 C CNN
@@
 $EndComp
 $Comp
-L +1.0V #PWR077
+L +1.0V #PWR076
 U 1 1 5479DBBA
 P 2975 4950
-F 0 "#PWR077" H 2975 5090 20  0001 C CNN
+F 0 "#PWR076" H 2975 5090 20  0001 C CNN
 F 1 "+1.0V" H 2975 5060 30  0000 C CNN
 F 2 "" H 2975 4950 60  0000 C CNN
@@
 $EndComp
 $Comp
-L +3,3V #PWR078
+L +3,3V #PWR077
 U 1 1 5479DBC0
 P 3000 2850
-F 0 "#PWR078" H 3000 2810 30  0001 C CNN
+F 0 "#PWR077" H 3000 2810 30  0001 C CNN
 F 1 "+3,3V" H 3000 2960 30  0000 C CNN
 F 2 "" H 3000 2850 60  0000 C CNN
@@
 $EndComp
 $Comp
-L DGND #PWR079
+L DGND #PWR078
 U 1 1 5479DC10
 P 4575 5325
-F 0 "#PWR079" H 4575 5325 40  0001 C CNN
+F 0 "#PWR078" H 4575 5325 40  0001 C CNN
 F 1 "DGND" H 4575 5255 40  0000 C CNN
 F 2 "" H 4575 5325 60  0000 C CNN
@@
 $EndComp
 $Comp
-L CP1 C60
+L CP1-RESCUE-preamp C60
 U 1 1 5479DC9A
 P 5600 2050
@@
 $EndComp
 $Comp
-L C C65
+L C-RESCUE-preamp C65
 U 1 1 5479DD06
 P 5825 2050
@@
 $EndComp
 $Comp
-L C C69
+L C-RESCUE-preamp C69
 U 1 1 5479DD3B
 P 6050 2050
@@
 $EndComp
 $Comp
-L C C73
+L C-RESCUE-preamp C73
 U 1 1 5479DDCF
 P 6275 2050
@@
 $EndComp
 $Comp
-L C C76
+L C-RESCUE-preamp C76
 U 1 1 5479DDD5
 P 6500 2050
@@
 $EndComp
 $Comp
-L C C79
+L C-RESCUE-preamp C79
 U 1 1 5479DE3F
 P 6725 2050
@@
 $EndComp
 $Comp
-L C C82
+L C-RESCUE-preamp C82
 U 1 1 5479DE45
 P 6950 2050
@@
 $EndComp
 $Comp
-L C C84
+L C-RESCUE-preamp C84
 U 1 1 5479DE5B
 P 7175 2050
@@
 $EndComp
 $Comp
-L C C85
+L C-RESCUE-preamp C85
 U 1 1 5479DEA8
 P 7400 2050
@@
 $EndComp
 $Comp
-L C C87
+L C-RESCUE-preamp C87
 U 1 1 5479DF36
 P 7625 2050
@@
 $EndComp
 $Comp
-L C C89
+L C-RESCUE-preamp C89
 U 1 1 5479DF3C
 P 7850 2050
@@
 $EndComp
 $Comp
-L C C91
+L C-RESCUE-preamp C91
 U 1 1 5479E082
 P 8075 2050
@@
 $EndComp
 $Comp
-L C C93
+L C-RESCUE-preamp C93
 U 1 1 5479E088
 P 8300 2050
@@
 $EndComp
 $Comp
-L C C95
+L C-RESCUE-preamp C95
 U 1 1 5479E08E
 P 8525 2050
@@
 $EndComp
 $Comp
-L C C97
+L C-RESCUE-preamp C97
 U 1 1 5479E094
 P 8750 2050
@@
 $EndComp
 $Comp
-L CP1 C61
+L CP1-RESCUE-preamp C61
 U 1 1 5479E0CA
 P 5600 2750
@@
 $EndComp
 $Comp
-L C C66
+L C-RESCUE-preamp C66
 U 1 1 5479E299
 P 5825 2750
@@
 $EndComp
 $Comp
-L C C70
+L C-RESCUE-preamp C70
 U 1 1 5479E29F
 P 6050 2750
@@
 $EndComp
 $Comp
-L C C62
+L C-RESCUE-preamp C62
 U 1 1 5479E2CB
 P 5600 3650
@@
 $EndComp
 $Comp
-L C C67
+L C-RESCUE-preamp C67
 U 1 1 5479E4AE
 P 5825 3650
@@
 $EndComp
 $Comp
-L C C71
+L C-RESCUE-preamp C71
 U 1 1 5479E4B4
 P 6050 3650
@@
 $EndComp
 $Comp
-L C C74
+L C-RESCUE-preamp C74
 U 1 1 5479E672
 P 6275 3650
@@
 $EndComp
 $Comp
-L C C77
+L C-RESCUE-preamp C77
 U 1 1 5479E678
 P 6500 3650
@@
 $EndComp
 $Comp
-L C C80
+L C-RESCUE-preamp C80
 U 1 1 5479E67E
 P 6725 3650
@@
 $EndComp
 $Comp
-L C C63
+L C-RESCUE-preamp C63
 U 1 1 5479E6B6
 P 5600 4450
@@
 $EndComp
 $Comp
-L C C64
+L C-RESCUE-preamp C64
 U 1 1 5479E716
 P 5600 5375
@@
 $EndComp
 $Comp
-L C C68
+L C-RESCUE-preamp C68
 U 1 1 5479E8BF
 P 6025 5375
@@
 $EndComp
 $Comp
-L C C72
+L C-RESCUE-preamp C72
 U 1 1 5479E8C5
 P 6250 5375
@@
 $EndComp
 $Comp
-L C C75
+L C-RESCUE-preamp C75
 U 1 1 5479EAC2
 P 6475 5375
@@
 $EndComp
 $Comp
-L C C78
+L C-RESCUE-preamp C78
 U 1 1 5479EAC8
 P 6700 5375
@@
 $EndComp
 $Comp
-L C C81
+L C-RESCUE-preamp C81
 U 1 1 5479EACE
 P 6925 5375
@@
 $EndComp
 $Comp
-L C C83
+L C-RESCUE-preamp C83
 U 1 1 5479EAD4
 P 7150 5375
@@
 $EndComp
 $Comp
-L +1.0V #PWR080
+L +1.0V #PWR079
 U 1 1 547A82BE
 P 5600 1750
-F 0 "#PWR080" H 5600 1890 20  0001 C CNN
+F 0 "#PWR079" H 5600 1890 20  0001 C CNN
 F 1 "+1.0V" H 5600 1860 30  0000 C CNN
 F 2 "" H 5600 1750 60  0000 C CNN
@@
 $EndComp
 $Comp
-L +1.0V #PWR081
+L +1.0V #PWR080
 U 1 1 547A85BD
 P 5600 2475
-F 0 "#PWR081" H 5600 2615 20  0001 C CNN
+F 0 "#PWR080" H 5600 2615 20  0001 C CNN
 F 1 "+1.0V" H 5600 2585 30  0000 C CNN
 F 2 "" H 5600 2475 60  0000 C CNN
@@
 $EndComp
 $Comp
-L +3,3V #PWR082
+L +3,3V #PWR081
 U 1 1 547A896F
 P 5600 4200
-F 0 "#PWR082" H 5600 4160 30  0001 C CNN
+F 0 "#PWR081" H 5600 4160 30  0001 C CNN
 F 1 "+3,3V" H 5600 4310 30  0000 C CNN
 F 2 "" H 5600 4200 60  0000 C CNN
@@
 $EndComp
 $Comp
-L +3,3V #PWR083
+L +3,3V #PWR082
 U 1 1 547A8A43
 P 5600 5075
-F 0 "#PWR083" H 5600 5035 30  0001 C CNN
+F 0 "#PWR082" H 5600 5035 30  0001 C CNN
 F 1 "+3,3V" H 5600 5185 30  0000 C CNN
 F 2 "" H 5600 5075 60  0000 C CNN
@@
 $EndComp
 $Comp
-L DGND #PWR084
+L DGND #PWR083
 U 1 1 547A8B87
 P 6725 4000
-F 0 "#PWR084" H 6725 4000 40  0001 C CNN
+F 0 "#PWR083" H 6725 4000 40  0001 C CNN
 F 1 "DGND" H 6725 3930 40  0000 C CNN
 F 2 "" H 6725 4000 60  0000 C CNN
@@
 $EndComp
 $Comp
-L DGND #PWR085
+L DGND #PWR084
 U 1 1 547A8BB3
 P 8750 2400
-F 0 "#PWR085" H 8750 2400 40  0001 C CNN
+F 0 "#PWR084" H 8750 2400 40  0001 C CNN
 F 1 "DGND" H 8750 2330 40  0000 C CNN
 F 2 "" H 8750 2400 60  0000 C CNN
@@
 $EndComp
 $Comp
-L DGND #PWR086
+L DGND #PWR085
 U 1 1 547AB50B
 P 5600 4750
-F 0 "#PWR086" H 5600 4750 40  0001 C CNN
+F 0 "#PWR085" H 5600 4750 40  0001 C CNN
 F 1 "DGND" H 5600 4680 40  0000 C CNN
 F 2 "" H 5600 4750 60  0000 C CNN
@@
 $EndComp
 $Comp
-L DGND #PWR087
+L DGND #PWR086
 U 1 1 547AB6A7
 P 6050 3150
-F 0 "#PWR087" H 6050 3150 40  0001 C CNN
+F 0 "#PWR086" H 6050 3150 40  0001 C CNN
 F 1 "DGND" H 6050 3080 40  0000 C CNN
 F 2 "" H 6050 3150 60  0000 C CNN
@@
 $EndComp
 $Comp
-L C C86
+L C-RESCUE-preamp C86
 U 1 1 547BA6F5
 P 7575 5375
@@
 $EndComp
 $Comp
-L C C88
+L C-RESCUE-preamp C88
 U 1 1 547BA6FB
 P 7800 5375
@@
 $EndComp
 $Comp
-L C C90
+L C-RESCUE-preamp C90
 U 1 1 547BA701
 P 8025 5375
@@
 $EndComp
 $Comp
-L C C92
+L C-RESCUE-preamp C92
 U 1 1 547BA707
 P 8250 5375
@@
 $EndComp
 $Comp
-L C C94
+L C-RESCUE-preamp C94
 U 1 1 547BA70D
 P 8475 5375
@@
 $EndComp
 $Comp
-L C C96
+L C-RESCUE-preamp C96
 U 1 1 547BA713
 P 8700 5375
@@
 $EndComp
 $Comp
-L DGND #PWR088
+L DGND #PWR087
 U 1 1 547BA71F
 P 8700 5750
-F 0 "#PWR088" H 8700 5750 40  0001 C CNN
+F 0 "#PWR087" H 8700 5750 40  0001 C CNN
 F 1 "DGND" H 8700 5680 40  0000 C CNN
 F 2 "" H 8700 5750 60  0000 C CNN
@@
 $EndComp
 $Comp
-L +1.8V #PWR089
+L +1.8V #PWR088
 U 1 1 548CD79C
 P 3125 2425
-F 0 "#PWR089" H 3125 2565 20  0001 C CNN
+F 0 "#PWR088" H 3125 2565 20  0001 C CNN
 F 1 "+1.8V" H 3125 2535 30  0000 C CNN
 F 2 "" H 3125 2425 60  0000 C CNN
@@
 $EndComp
 $Comp
-L +1.8V #PWR090
+L +1.8V #PWR089
 U 1 1 548CE474
 P 5600 3325
-F 0 "#PWR090" H 5600 3465 20  0001 C CNN
+F 0 "#PWR089" H 5600 3465 20  0001 C CNN
 F 1 "+1.8V" H 5600 3435 30  0000 C CNN
 F 2 "" H 5600 3325 60  0000 C CNN
@@
 	3200 1725 3200 1825
 $Comp
-L DGND #PWR091
+L DGND #PWR090
 U 1 1 549497E2
 P 3075 4300
-F 0 "#PWR091" H 3075 4300 40  0001 C CNN
+F 0 "#PWR090" H 3075 4300 40  0001 C CNN
 F 1 "DGND" H 3075 4230 40  0000 C CNN
 F 2 "" H 3075 4300 60  0000 C CNN
