File: asd_pre_1/pcb/power.sch (KiCad schematic (older format))
At the start: 46 parts, among them P5 PwGnd, U10 LM2937-12, U11 L79L12, U12 TPS54325, U13 TPS54294, U14 L78L05

Commit message: Updated schematics and PCB.  Removed some minor errors with the first prototype.
Parts:
- C100, C101, C102, C104, C105, C106, C107, C108, C109, C110, C111, C112, C113, C114, C115, C116, C117, C118, C119, C120, C121, C122, C123, C124, C125, C126, C98, C99: symbol C -> C-RESCUE-preamp
- C103: symbol CP1 -> CP1-RESCUE-preamp
- R46, R47, R48, R49, R50, R51, R52, R53: symbol R -> R-RESCUE-preamp
Changed lines of the file:
@@
 EESchema Schematic File Version 2
+LIBS:preamp-rescue
 LIBS:power
 LIBS:device
@@
 LIBS:memory
 LIBS:xilinx
-LIBS:special
 LIBS:microcontrollers
 LIBS:dsp
@@
 encoding utf-8
 Sheet 8 9
-Title ""
+Title "AsD Pre 1 Digital Preamplifier -- Power"
 Date ""
 Rev ""
-Comp ""
+Comp "Asbjørn Djupdal"
 Comment1 ""
 Comment2 ""
@@
 $EndDescr
 $Comp
-L +3,3V #PWR092
+L +3,3V #PWR091
 U 1 1 546883B2
 P 9050 4775
-F 0 "#PWR092" H 9050 4735 30  0001 C CNN
+F 0 "#PWR091" H 9050 4735 30  0001 C CNN
 F 1 "+3,3V" H 9050 4885 30  0000 C CNN
 F 2 "" H 9050 4775 60  0000 C CNN
@@
 $EndComp
 $Comp
-L +5VA #PWR093
+L +5VA #PWR092
 U 1 1 546883DA
 P 7025 1300
-F 0 "#PWR093" H 7025 1430 20  0001 C CNN
+F 0 "#PWR092" H 7025 1430 20  0001 C CNN
 F 1 "+5VA" H 7025 1400 30  0000 C CNN
 F 2 "" H 7025 1300 60  0000 C CNN
@@
 $EndComp
 $Comp
-L AGND #PWR094
-U 1 1 546883EE
-P 3025 2600
-F 0 "#PWR094" H 3025 2600 40  0001 C CNN
-F 1 "AGND" H 3025 2530 50  0000 C CNN
-F 2 "" H 3025 2600 60  0000 C CNN
-F 3 "" H 3025 2600 60  0000 C CNN
-	1    3025 2600
-	1    0    0    -1
-$EndComp
-$Comp
-L DGND #PWR095
+L DGND #PWR093
 U 1 1 54688402
 P 3250 2050
-F 0 "#PWR095" H 3250 2050 40  0001 C CNN
+F 0 "#PWR093" H 3250 2050 40  0001 C CNN
 F 1 "DGND" H 3250 1980 40  0000 C CNN
 F 2 "" H 3250 2050 60  0000 C CNN
@@
 $EndComp
 $Comp
-L +VOA #PWR096
+L +VOA #PWR094
 U 1 1 546877F7
 P 5700 1300
-F 0 "#PWR096" H 5700 1430 20  0001 C CNN
+F 0 "#PWR094" H 5700 1430 20  0001 C CNN
 F 1 "+VOA" H 5700 1400 30  0000 C CNN
 F 2 "" H 5700 1300 60  0000 C CNN
@@
 $EndComp
 $Comp
-L -VOA #PWR097
+L -VOA #PWR095
 U 1 1 5468780B
 P 6375 2250
-F 0 "#PWR097" H 6375 2380 20  0001 C CNN
+F 0 "#PWR095" H 6375 2380 20  0001 C CNN
 F 1 "-VOA" H 6375 2350 30  0000 C CNN
 F 2 "" H 6375 2250 60  0000 C CNN
@@
 $EndComp
 $Comp
-L C C107
+L C-RESCUE-preamp C107
 U 1 1 548A0291
 P 4575 2100
@@
 $EndComp
 $Comp
-L C C109
+L C-RESCUE-preamp C109
 U 1 1 548A033A
 P 5575 2100
@@
 $EndComp
 $Comp
-L C C108
+L C-RESCUE-preamp C108
 U 1 1 548A037D
 P 5575 1650
@@
 $EndComp
 $Comp
-L C C106
+L C-RESCUE-preamp C106
 U 1 1 548A03C9
 P 4575 1650
@@
 $EndComp
 $Comp
-L C C111
+L C-RESCUE-preamp C111
 U 1 1 548A0430
 P 5825 1650
@@
 $EndComp
 $Comp
-L C C117
+L C-RESCUE-preamp C117
 U 1 1 548A04A8
 P 6750 1650
@@
 $EndComp
 $Comp
-L C C101
+L C-RESCUE-preamp C101
 U 1 1 548B1272
 P 3225 3025
@@
 $EndComp
 $Comp
-L C C102
+L C-RESCUE-preamp C102
 U 1 1 548B141F
 P 3450 3025
@@
 $EndComp
 $Comp
-L CP1 C103
+L CP1-RESCUE-preamp C103
 U 1 1 548B2224
 P 3575 1425
@@
 $EndComp
 $Comp
-L R R48
+L R-RESCUE-preamp R48
 U 1 1 548B27D8
 P 3800 3250
@@
 $EndComp
 $Comp
-L R R49
+L R-RESCUE-preamp R49
 U 1 1 548B2899
 P 3800 3800
@@
 $EndComp
 $Comp
-L C C105
+L C-RESCUE-preamp C105
 U 1 1 548B2FF6
 P 4100 3575
@@
 $EndComp
 $Comp
-L C C110
+L C-RESCUE-preamp C110
 U 1 1 548B31E1
 P 5800 3525
@@
 $EndComp
 $Comp
-L R R50
+L R-RESCUE-preamp R50
 U 1 1 548B335B
 P 6150 3325
@@
 $EndComp
 $Comp
-L C C115
+L C-RESCUE-preamp C115
 U 1 1 548B3632
 P 6475 2975
@@
 $EndComp
 $Comp
-L C C122
+L C-RESCUE-preamp C122
 U 1 1 548B3B29
 P 7500 3075
@@
 $EndComp
 $Comp
-L C C123
+L C-RESCUE-preamp C123
 U 1 1 548B3C0A
 P 7725 3075
@@
 $EndComp
 $Comp
-L +1.0V #PWR098
+L +1.0V #PWR096
 U 1 1 548B3EC6
 P 7975 2725
-F 0 "#PWR098" H 7975 2865 20  0001 C CNN
+F 0 "#PWR096" H 7975 2865 20  0001 C CNN
 F 1 "+1.0V" H 7975 2835 30  0000 C CNN
 F 2 "" H 7975 2725 60  0000 C CNN
@@
 $EndComp
 $Comp
-L C C114
+L C-RESCUE-preamp C114
 U 1 1 548B9BFD
 P 6450 4700
@@
 $EndComp
 $Comp
-L C C116
+L C-RESCUE-preamp C116
 U 1 1 548B9D3F
 P 6675 4700
@@
 $EndComp
 $Comp
-L C C118
+L C-RESCUE-preamp C118
 U 1 1 548B9D88
 P 6900 4700
@@
 $EndComp
 $Comp
-L C C120
+L C-RESCUE-preamp C120
 U 1 1 548B9E18
 P 7125 4700
@@
 $EndComp
 $Comp
-L C C104
+L C-RESCUE-preamp C104
 U 1 1 548BB3C8
 P 4075 5200
@@
 $EndComp
 $Comp
-L C C100
+L C-RESCUE-preamp C100
 U 1 1 548BB846
 P 3075 5200
@@
 $EndComp
 $Comp
-L C C99
+L C-RESCUE-preamp C99
 U 1 1 548BB90B
 P 2875 5200
@@
 $EndComp
 $Comp
-L R R46
+L R-RESCUE-preamp R46
 U 1 1 548BBC89
 P 2650 5250
@@
 $EndComp
 $Comp
-L R R47
+L R-RESCUE-preamp R47
 U 1 1 548BBD49
 P 2650 5800
@@
 $EndComp
 $Comp
-L C C98
+L C-RESCUE-preamp C98
 U 1 1 548BCF06
 P 2350 5250
@@
 $EndComp
 $Comp
-L C C113
+L C-RESCUE-preamp C113
 U 1 1 548BD172
 P 5975 5750
@@
 Wire Wire Line
 	3250 1050 3250 2050
-Wire Wire Line
-	3025 1875 3025 2600
 Connection ~ 4575 1425
 Wire Wire Line
@@
 	3575 1225 3575 950
 Connection ~ 3575 950
-Wire Wire Line
-	3575 1875 3575 1625
 Connection ~ 3575 1875
 Connection ~ 3450 2825
@@
 Connection ~ 6150 3050
 $Comp
-L R R51
+L R-RESCUE-preamp R51
 U 1 1 548BDE00
 P 6450 5775
@@
 Connection ~ 6450 6175
 $Comp
-L +1.8V #PWR099
+L +1.8V #PWR097
 U 1 1 548BEE7A
 P 2350 4775
-F 0 "#PWR099" H 2350 4915 20  0001 C CNN
+F 0 "#PWR097" H 2350 4915 20  0001 C CNN
 F 1 "+1.8V" H 2350 4885 30  0000 C CNN
 F 2 "" H 2350 4775 60  0000 C CNN
@@
 $EndComp
 $Comp
-L C C121
+L C-RESCUE-preamp C121
 U 1 1 548C09A4
 P 7300 5200
@@
 $EndComp
 $Comp
-L C C124
+L C-RESCUE-preamp C124
 U 1 1 548C09AA
 P 8325 5200
@@
 $EndComp
 $Comp
-L C C125
+L C-RESCUE-preamp C125
 U 1 1 548C09B0
 P 8525 5200
@@
 $EndComp
 $Comp
-L R R52
+L R-RESCUE-preamp R52
 U 1 1 548C09B7
 P 8750 5250
@@
 $EndComp
 $Comp
-L R R53
+L R-RESCUE-preamp R53
 U 1 1 548C09BE
 P 8750 5800
@@
 $EndComp
 $Comp
-L C C126
+L C-RESCUE-preamp C126
 U 1 1 548C09C4
 P 9050 5250
@@
 	4425 1150 2300 1150
 Wire Wire Line
-	3025 1875 7025 1875
-Wire Wire Line
 	3250 1050 2300 1050
 Connection ~ 3250 1875
@@
 Connection ~ 4075 5400
 $Comp
-L C C119
+L C-RESCUE-preamp C119
 U 1 1 5496F9A0
 P 7025 1650
@@
 $EndComp
 $Comp
-L C C112
+L C-RESCUE-preamp C112
 U 1 1 5496FBC7
 P 5825 2100
@@
 Connection ~ 5825 2325
 $Comp
-L +3.3VDAC #PWR0100
+L +3.3VDAC #PWR098
 U 1 1 54A031C7
 P 9925 4775
-F 0 "#PWR0100" H 9925 4895 20  0001 C CNN
+F 0 "#PWR098" H 9925 4895 20  0001 C CNN
 F 1 "+3.3VDAC" H 9925 4865 30  0000 C CNN
 F 2 "" H 9925 4775 60  0000 C CNN
@@
 Wire Wire Line
 	9925 5000 9925 4775
+Wire Wire Line
+	3025 1875 7025 1875
+Wire Wire Line
+	3575 1625 3575 2050
+Text GLabel 3025 1875 0    60   Input ~ 0
+DGND
+$Comp
+L AGND #PWR?
+U 1 1 58E2BA30
+P 3575 2050
+F 0 "#PWR?" H 3575 2050 40  0001 C CNN
+F 1 "AGND" H 3575 1980 50  0000 C CNN
+F 2 "" H 3575 2050 60  0000 C CNN
+F 3 "" H 3575 2050 60  0000 C CNN
+	1    3575 2050
+	1    0    0    -1
+$EndComp
 $EndSCHEMATC
