File: asd_pre_1/pcb/spdif.sch (KiCad schematic (older format))
At the start: 18 parts, among them P3 TOSLINK, P4 SPDIF, T1 S22083, U2 MAX3280E, U3 DIR9001

Commit message: Updated schematics and PCB.  Removed some minor errors with the first prototype.
Parts:
- C13, C15, C16, C17, C19, C20: symbol C -> C-RESCUE-preamp
- C14, C18: symbol CP1 -> CP1-RESCUE-preamp
- R13, R14, R15: symbol R -> R-RESCUE-preamp
Changed lines of the file:
@@
 EESchema Schematic File Version 2
+LIBS:preamp-rescue
 LIBS:power
 LIBS:device
@@
 LIBS:memory
 LIBS:xilinx
-LIBS:special
 LIBS:microcontrollers
 LIBS:dsp
@@
 encoding utf-8
 Sheet 3 9
-Title ""
+Title "AsD Pre 1 Digital Preamplifier -- SPDIF"
 Date ""
 Rev ""
-Comp ""
+Comp "Asbjørn Djupdal"
 Comment1 ""
 Comment2 ""
@@
 $EndComp
 $Comp
-L CP1 C14
+L CP1-RESCUE-preamp C14
 U 1 1 54653476
 P 3300 4475
@@
 $EndComp
 $Comp
-L C C15
+L C-RESCUE-preamp C15
 U 1 1 546534F9
 P 3600 4475
@@
 $EndComp
 $Comp
-L CP1 C18
+L CP1-RESCUE-preamp C18
 U 1 1 5465379A
 P 6750 4475
@@
 $EndComp
 $Comp
-L C C17
+L C-RESCUE-preamp C17
 U 1 1 54653834
 P 6500 4475
@@
 $EndComp
 $Comp
-L C C16
+L C-RESCUE-preamp C16
 U 1 1 54653A31
 P 6275 5425
@@
 $EndComp
 $Comp
-L C C19
+L C-RESCUE-preamp C19
 U 1 1 54653AC9
 P 6825 5425
@@
 $EndComp
 $Comp
-L R R15
+L R-RESCUE-preamp R15
 U 1 1 54653B1D
 P 6550 5625
@@
 $EndComp
 $Comp
-L R R14
+L R-RESCUE-preamp R14
 U 1 1 54653FF7
 P 5975 4825
@@
 $EndComp
 $Comp
-L C C20
+L C-RESCUE-preamp C20
 U 1 1 546650C1
 P 9150 2000
@@
 $EndComp
 $Comp
-L R R13
+L R-RESCUE-preamp R13
 U 1 1 54666390
 P 4350 1800
@@
 $EndComp
 $Comp
-L C C13
+L C-RESCUE-preamp C13
 U 1 1 54667021
 P 2775 1325
